File: FT2232H_EVB.kicad_sch (KiCad schematic)
At the start: 193 parts, among them IC1 MT9700, IC2 SL2.1s, IC3 W25Q16JVUXIQ, IC4 LCMXO2-1200HC-4SG32I, J1 GT-USB-7010ASV, J11 Conn_02x03_Odd_Even, J2 WJ126V-5.0-2P, J3 WJ126V-5.0-2P, J4 WJ126V-5.0-2P, J5 WJ126V-5.0-2P, J6 Conn_01x04, J6 Conn_02x03_Odd_Even, J7 Conn_02x03_Odd_Even, J8 Conn_02x03_Odd_Even, J9 Conn_02x03_Odd_Even, SW1 DSWB03LHGET, U1 RT5752AHGJ5, U2 TLV803SDBZR, U3 RQ12000160, U4 ADS1115IDGSR, U5 RP2040, U7 ADS1115IDGSR, U8 FT2232HL, U8 RQ12000160, U9 93LC56BT-I, U9 RQ12000160

Commit message: first commit
Parts:
- removed C74, C77: 0.1uF, Capacitor_SMD:C_0201_0603Metric_Pad0.64x0.40mm_HandSolder, symbol Device:C_Small
- removed R38: 10k, Resistor_SMD:R_0201_0603Metric_Pad0.64x0.40mm_HandSolder, symbol Device:R
- removed R67, R68, R69: 1k, Resistor_SMD:R_0201_0603Metric_Pad0.64x0.40mm_HandSolder, symbol Device:R
- removed TP1, TP6, TP8: TestPoint, TestPoint:TestPoint_Pad_D1.0mm, symbol Connector:TestPoint
- removed U1: RT5752AHGJ5, Package_TO_SOT_SMD:TSOT-23-5, symbol RT5752AHGJ5:RT5752AHGJ5
- removed U4, U7: ADS1115IDGSR, ADS1115IDGSR:DGS0010A_M, symbol ADS1115IDGSR:ADS1115IDGSR
- added C82, C83: 0.1uF, Capacitor_SMD:C_0201_0603Metric_Pad0.64x0.40mm_HandSolder, symbol Device:C_Small
- added J13: Conn_02x01, Connector_PinHeader_2.54mm:PinHeader_2x01_P2.54mm_Vertical, symbol Connector_Generic:Conn_02x01
- added L5, L9: HCB1005KF-121T20, Resistor_SMD:R_0402_1005Metric_Pad0.72x0.64mm_HandSolder, symbol hcb1005kf-121t20:HCB1005KF-121T20
- added U1: RT5752BHGJ5, Package_TO_SOT_SMD:TSOT-23-5, symbol RT5752BHGJ5:RT5752BHGJ5
- added U4, U7: ADS1118IDGSR, ADS1118IDGSR:DGS0010A_M, symbol ADS1118IDGSR:ADS1118IDGSR
- R12: value 0 -> 30
- R3: value 3.4k -> 3.6k; footprint Resistor_SMD:R_0402_1005Metric_Pad0.72x0.64mm_HandSolder -> Resistor_SMD:R_0201_0603Metric_Pad0.64x0.40mm_HandSolder
- R54, R57, R58: value 0 -> 10k
- R60: value 0 -> 10k; now fitted
- R66: value 1k -> 10k
- R9: value 2.2k -> 30
Connections:
- net I2CSCL_ADC is gone; now on net I2CSCL_EXT: R17.2, U5.5 (GPIO3)
- net I2CSDA_ADC is gone; now on net I2CSDA_EXT: R18.2, U5.4 (GPIO2)
- net +3.3V: now also C82.1, L5.1
- net +3.3V_ADC: now also R23.1, R54.1, R57.1, R58.1, R60.1, R66.1, U4.8 (VDD), U7.8 (VDD)
- net ADC0(GPIO26): now also J11.4 (Pin_4); no longer C75.1, R66.1
- net GND: now also C82.2, C83.2, J13.2 (Pin_2), U1.2 (GND), U4.3 (GND), U7.3 (GND); no longer R23.2
- net TDI/SWDIO_PIN: now also J8.3 (Pin_3); no longer R57.1
- net TDO_PIN: now also J8.4 (Pin_4); no longer R58.1, R60.2
- net TMS_PIN: now also J8.2 (Pin_2); no longer R54.1
- net VBUS: now also L9.1
- net at C53.1, C54.2, R39.2: now also U7.4 (AIN0)
- net at C54.1, C55.1, R40.2: now also U7.5 (AIN1)
- net at C65.1, C66.2, R43.2: now also U7.6 (AIN2)
- net at C66.1, C67.1, R44.2: now also U7.7 (AIN3)
- net SPI1_MOSI: now reaches U5.14 (GPIO11)
- net SPI1_MOSI: now also R54.2, R58.2, U4.10 (DIN), U7.10 (DIN)
- net I2CSDA_EXT: now reaches J11.2 (Pin_2)
- net SPI1_CS0_N: now reaches U5.6 (GPIO4)
- net SPI1_CS0_N: now also R57.2, U4.2 (CS_N)
- net at C2.1, IC1.5 (VIN), L1.2: now also IC1.4 (EN); no longer IC1.3 (SET)
- net at C8.1, R4.1, R8.2: now also U1.5 (FB)
- net at C18.1, U3.3 (OSC2): now also IC2.11 (XOUT); no longer R12.2
- net at C49.1, C50.1, R33.2: now also U4.7 (AIN3)
- net at C3.1, C4.1, L2.2: now also U1.1 (EN), U1.4 (VIN)
- net at L3.1: now also U1.3 (SW)
- net at C35.1, C36.2, R19.2: now also U4.4 (AIN0)
- net at C36.1, C45.1, R20.2: now also U4.5 (AIN1)
- net at C46.1, C49.2, R31.2: now also U4.6 (AIN2)
- net SPI1_MISO: now reaches U5.11 (GPIO8)
- net SPI1_MISO: now also R23.2, R60.2, U4.9 (DOUT/DRDY_N), U7.9 (DOUT/DRDY_N)
- net at U5.13 (GPIO10): now also R12.1
- net SPI1_CS1_N: now reaches U5.36 (GPIO24)
- net SPI1_CS1_N: now also R66.2, U7.2 (CS_N)
- net at R3.1: now also IC1.3 (SET); no longer IC1.4 (EN)
- net +3.3V_EXT: now reaches J11.3 (Pin_3)
- net +3.3V_EXT: now also C76.1, C83.1, L5.2
- net I2CSCL_EXT: now reaches J11.1 (Pin_1)
- net I2CSCL_EXT: no longer R66.2
- net ADC1(GPIO27): no longer names the net of U5.39 (GPIO27_ADC1)
- net ADC1(GPIO27): no longer C76.1
- net ADC2(GPIO28): no longer names the net of U5.40 (GPIO28_ADC2)
- net ADC3(GPIO28): no longer names the net of U5.41 (GPIO29_ADC3)
- new net SPI1_CLK0: R12.2, U4.1 (SCLK), U7.1 (SCLK)
- new net VBUS_EXT: C75.1, J13.1 (Pin_1), L9.2
- no-connect marks 43 -> 42
Other:
- note added: "500mAmax"
- note added: "Current Limit 1.9A(Rset=3.6kΩ)"
- note added: "External Power Pinheader"
- note added: "External Signal Pinheader"
- note added: "R12はU5の直近に配置"
- note added: "R12ランド直後に分岐(スタブ注意) SPI1_CLK0とSPI1_CLK1は 可能な限り等長配線"
- note added: "min:3.24V typ:3.33V max:3.42V 0.647Amax"
- note removed: "0Ω"
- note removed: "470Ω"
- note removed: "ADC Pinheader"
- note removed: "Current Limit 2A(Rset=3.4kΩ)"
- note removed: "OPEN"
- note removed: "R54"
- note removed: "R57"
- note removed: "R58"
- note removed: "R60"
- note removed: "SLAVE ADDRESS 1001000"
- note removed: "SLAVE ADDRESS 1001001"
- note removed: "SWD"
- note removed: "min:3.24V typ:3.33V max:3.42V 1.087Amax"
- moved on the sheet: R23

Commit message: 3S commit
Parts:
- renumbered C6 to C1, C33 to C73, D7 to D1, D6 to D2, J6 to J10, R3 to R7, U9 to U10, U8 to U6
Connections:
- net ADC0(GPIO26) renamed EVBDET_N
