File: FT2232H_EVB.kicad_sch (KiCad schematic)
At the start: 209 parts, among them IC1 MT9700, IC2 SL2.1s, IC3 W25Q16JVUXIQ, IC4 LCMXO2-1200HC-4SG32I, J1 GT-USB-7010ASV, J10 Conn_01x04, J11 Conn_02x03_Odd_Even, J13 Conn_02x01, J2 WJ126V-5.0-2P, J3 WJ126V-5.0-2P, J4 WJ126V-5.0-2P, J5 WJ126V-5.0-2P, J6 Conn_02x03_Odd_Even, J7 Conn_02x03_Odd_Even, J8 Conn_02x03_Odd_Even, J9 Conn_02x03_Odd_Even, SW1 DSWB03LHGET, U1 RT5752BHGJ5, U10 RQ12000160, U2 TLV803SDBZR, U3 RQ12000160, U4 ADS1118IDGSR, U5 RP2040, U6 RQ12000160, U7 ADS1118IDGSR, U8 FT2232HL, U9 93LC56BT-I

Commit message: Mass Production2 commit
Parts:
- removed C8: 10p, Capacitor_SMD:C_0201_0603Metric_Pad0.64x0.40mm_HandSolder, symbol Device:C_Small
Changed lines of the file:
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@@
 	)
 	(junction
-		(at 221.869 40.767)
-		(diameter 0)
-		(color 0 0 0 0)
-	)
-	(junction
 		(at 510.667 107.188)
 		(diameter 0)
@@
 	)
 	(junction
-		(at 207.391 44.323)
-		(diameter 0)
-		(color 0 0 0 0)
-	)
-	(junction
 		(at 18.161 94.869)
 		(diameter 0)
@@
 	(wire
 		(pts
-			(xy 207.391 44.323) (xy 211.709 44.323)
-		)
-		(stroke
-			(width 0)
-			(type default)
-		)
-	)
-	(wire
-		(pts
 			(xy 134.62 160.528) (xy 135.509 160.528)
 		)
@@
 	(wire
 		(pts
-			(xy 207.391 44.323) (xy 207.391 45.085)
+			(xy 207.391 40.767) (xy 207.391 45.085)
 		)
 		(stroke
@@
 	(wire
 		(pts
-			(xy 216.789 44.323) (xy 221.869 44.323)
-		)
-		(stroke
-			(width 0)
-			(type default)
-		)
-	)
-	(wire
-		(pts
 			(xy 66.294 346.456) (xy 67.183 346.456)
 		)
@@
 	(wire
 		(pts
-			(xy 207.391 40.767) (xy 207.391 44.323)
-		)
-		(stroke
-			(width 0)
-			(type default)
-		)
-	)
-	(wire
-		(pts
 			(xy 374.142 266.065) (xy 374.142 285.623)
 		)
@@
 	(wire
 		(pts
-			(xy 221.869 44.323) (xy 221.869 40.767)
-		)
-		(stroke
-			(width 0)
-			(type default)
-		)
-	)
-	(wire
-		(pts
 			(xy 83.312 85.979) (xy 83.312 74.549)
 		)
@@
 					(unit 1)
 				)
-			)
-		)
-	)
-	(symbol
-		(lib_id "Device:C_Small")
-		(at 214.249 44.323 90)
-		(unit 1)
-		(exclude_from_sim no)
-		(in_bom yes)
-		(on_board yes)
-		(dnp yes)
-		(property "Reference" "C8"
-			(at 211.963 43.307 90)
-			(effects
-				(font
-					(size 1.27 1.27)
-				)
-				(justify left)
-			)
-		)
-		(property "Value" "10p"
-			(at 220.853 43.307 90)
-			(effects
-				(font
-					(size 1.27 1.27)
-				)
-				(justify left)
-			)
-		)
-		(property "Footprint" "Capacitor_SMD:C_0201_0603Metric_Pad0.64x0.40mm_HandSolder"
-			(at 214.249 44.323 0)
-			(effects
-				(font
-					(size 1.27 1.27)
-				)
-				(hide yes)
-			)
-		)
-		(property "Datasheet" "~"
-			(at 214.249 44.323 0)
-			(effects
-				(font
-					(size 1.27 1.27)
-				)
-				(hide yes)
-			)
-		)
-		(property "Description" "Unpolarized capacitor, small symbol"
-			(at 214.249 44.323 0)
-			(effects
-				(font
-					(size 1.27 1.27)
-				)
-				(hide yes)
-			)
-		)
-		(pin "1"
-		)
-		(pin "2"
-		)
-		(instances
-			(project "FT2232H_EVB"
-				(path "/483d0913-2604-458a-955b-5458dee34109"
-					(reference "C8")
-					(unit 1)
-				)

Commit message: Mass Production2 commit
Parts:
- removed R62: 0, Resistor_SMD:R_0201_0603Metric_Pad0.64x0.40mm_HandSolder, symbol Device:R
- S1: footprint SW_SKRPACE010 -> SKRPACE010:SW_SKRPACE010
Connections:
- net at U8.3 (OSCO): now also C73.1, R65.2, U10.3 (OSC2)
Changed lines of the file:
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@@
 	(wire
 		(pts
-			(xy 275.971 371.983) (xy 276.225 371.983)
-		)
-		(stroke
-			(width 0)
-			(type default)
-		)
-	)
-	(wire
-		(pts
 			(xy 91.059 147.828) (xy 104.14 147.828)
 		)
@@
 	(wire
 		(pts
-			(xy 268.351 371.983) (xy 265.303 371.983)
+			(xy 265.303 371.983) (xy 276.225 371.983)
 		)
 		(stroke
@@
 			)
 		)
-		(property "Footprint" "SW_SKRPACE010"
+		(property "Footprint" "SKRPACE010:SW_SKRPACE010"
 			(at 447.675 62.103 0)
 			(effects
@@
 					(unit 1)
 				)
-			)
-		)
-	)
-	(symbol
-		(lib_id "Device:R")
-		(at 272.161 371.983 90)
-		(unit 1)
-		(exclude_from_sim no)
-		(in_bom yes)
-		(on_board yes)
-		(dnp no)
-		(property "Reference" "R62"
-			(at 268.859 370.713 90)
-			(effects
-				(font
-					(size 1.27 1.27)
-				)
-				(justify left)
-			)
-		)
-		(property "Value" "0"
-			(at 272.923 371.983 90)
-			(effects
-				(font
-					(size 1.27 1.27)
-				)
-				(justify left)
-			)
-		)
-		(property "Footprint" "Resistor_SMD:R_0201_0603Metric_Pad0.64x0.40mm_HandSolder"
-			(at 272.161 373.761 90)
-			(effects
-				(font
-					(size 1.27 1.27)
-				)
-				(hide yes)
-			)
-		)
-		(property "Datasheet" "~"
-			(at 272.161 371.983 0)
-			(effects
-				(font
-					(size 1.27 1.27)
-				)
-				(hide yes)
-			)
-		)
-		(property "Description" "0201WMF0000TEE"
-			(at 272.161 371.983 0)
-			(effects
-				(font
-					(size 1.27 1.27)
-				)
-				(hide yes)
-			)
-		)
-		(property "耐電力" "1/20W"
-			(at 272.161 374.396 90)
-			(effects
-				(font
-					(size 1.016 1.016)
-				)
-			)
-		)
-		(pin "1"
-		)
-		(pin "2"
-		)
-		(instances
-			(project "FT2232H_EVB"
-				(path "/483d0913-2604-458a-955b-5458dee34109"
-					(reference "R62")
-					(unit 1)
-				)

Commit message: Mass Production2 commit
Parts:
- J13: value Conn_02x01 -> PH-2A; footprint Connector_PinHeader_2.54mm:PinHeader_2x01_P2.54mm_Vertical -> Connector_JST:JST_PH_B2B-PH-K_1x02_P2.00mm_Vertical
Changed lines of the file:
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@@
 			)
 		)
-		(property "Value" "Conn_02x01"
+		(property "Value" "PH-2A"
 			(at 49.149 369.951 0)
 			(effects
@@
 			)
 		)
-		(property "Footprint" "Connector_PinHeader_2.54mm:PinHeader_2x01_P2.54mm_Vertical"
+		(property "Footprint" "Connector_JST:JST_PH_B2B-PH-K_1x02_P2.00mm_Vertical"
 			(at 48.006 367.411 0)
 			(effects
