File: FT2232H_EVB.kicad_pcb (KiCad board)
At the start: 6 copper layers, 50 x 50 mm, 198 parts, among them IC1 MT9700, IC2 SL2.1s, IC3 W25Q16JVUXIQ, IC4 LCMXO2-1200HC-4SG32I, J1 GT-USB-7010ASV, J10 Conn_01x04, J11 Conn_02x03_Odd_Even, J2 WJ126V-5.0-2P, J3 WJ126V-5.0-2P, J4 WJ126V-5.0-2P, J5 WJ126V-5.0-2P, J6 Conn_02x03_Odd_Even, J7 Conn_02x03_Odd_Even, J8 Conn_02x03_Odd_Even, J9 Conn_02x03_Odd_Even, SW1 DSWB03LHGET, U1 RT5752AHGJ5, U10 RQ12000160, U11 TMUX1574DYYR, U12 TMUX1574DYYR, U2 TLV803SDBZR, U3 RQ12000160, U4 ADS1115IDGSR, U5 RP2040, U6 RQ12000160, U7 ADS1115IDGSR, U8 FT2232HL, U9 SOT-23-6

Commit message: first commit
Parts:
- removed C74, C77: 0.1uF, Capacitor_SMD:C_0201_0603Metric_Pad0.64x0.40mm_HandSolder
- removed R38: 10k, Resistor_SMD:R_0201_0603Metric_Pad0.64x0.40mm_HandSolder
- removed R67, R68, R69: 1k, Resistor_SMD:R_0201_0603Metric_Pad0.64x0.40mm_HandSolder
- removed TP1, TP6, TP8: TestPoint, TestPoint:TestPoint_Pad_D1.0mm
- added C82: 0.1uF, Capacitor_SMD:C_0201_0603Metric_Pad0.64x0.40mm_HandSolder, B.Cu at (129.7, 91.3)
- added C83: 0.1uF, Capacitor_SMD:C_0201_0603Metric_Pad0.64x0.40mm_HandSolder, B.Cu at (129.6, 88.3)
- added J13: Conn_02x01, Connector_PinHeader_2.54mm:PinHeader_2x01_P2.54mm_Vertical, F.Cu at (113.5, 84.3)
- added L5: HCB1005KF-121T20, Resistor_SMD:R_0402_1005Metric_Pad0.72x0.64mm_HandSolder, B.Cu at (129.2, 89.8)
- added L9: HCB1005KF-121T20, Resistor_SMD:R_0402_1005Metric_Pad0.72x0.64mm_HandSolder, B.Cu at (127.4, 105.2)
- R12: value 0 -> 30
- R54, R57, R58, R60: value 0 -> 10k
- R66: value 1k -> 10k
- R7: value 3.4k -> 3.6k; footprint Resistor_SMD:R_0402_1005Metric_Pad0.72x0.64mm_HandSolder -> Resistor_SMD:R_0201_0603Metric_Pad0.64x0.40mm_HandSolder
- R9: value 2.2k -> 30
- U1: value RT5752AHGJ5 -> RT5752BHGJ5
- U4, U7: value ADS1115IDGSR -> ADS1118IDGSR; footprint ADS1115IDGSR:DGS0010A_M -> ADS1118IDGSR:DGS0010A_M
- U9: value SOT-23-6 -> 93LC56BT-I
- moved R57 51.1 mm to (124.3, 79.9)
- moved R66 40.3 mm to (145.5, 79.9)
- moved R54 37.6 mm to (133.5, 82.2), turned to 180 degrees
- moved R60 32.5 mm to (154.7, 81.4), turned to 180 degrees
- moved C75 31.9 mm to (114.7, 82.9), turned to 0 degrees
- moved R58 31.7 mm to (154.7, 82.2), turned to 180 degrees
- moved R12 13.3 mm to (133.5, 110.0), turned to 180 degrees
- moved R23 9.40 mm to (133.5, 81.4)
- moved C76 8.57 mm to (128.2, 113.7), turned to 0 degrees
- moved C35 4.91 mm to (122.7, 74.7), turned to 90 degrees
- moved C67 4.84 mm to (156.7, 74.8), turned to 90 degrees
- moved C45 4.74 mm to (124.4, 74.7), turned to 90 degrees
- moved C65 4.69 mm to (154.9, 74.8), turned to 90 degrees
- moved C46 4.69 mm to (133.4, 74.8), turned to 90 degrees
- moved C53 4.67 mm to (144.2, 74.8), turned to 90 degrees
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Connections:
- C18 pad 1: Net-(U3-OSC2) -> Net-(IC2-XOUT)
- C2 pad 1: Net-(IC1-SET) -> Net-(IC1-EN)
- C75 pad 1: ADC0(GPIO26) -> VBUS_EXT
- C76 pad 1: ADC1(GPIO27) -> +3.3V_EXT
- IC1 pad 5: Net-(IC1-SET) -> Net-(IC1-EN)
- J11 pad 1: Net-(J11-Pin_1) -> I2CSCL_EXT
- J11 pad 2: Net-(J11-Pin_2) -> I2CSDA_EXT
- J11 pad 3: Net-(J11-Pin_3) -> +3.3V_EXT
- J11 pad 4: Net-(J11-Pin_4) -> ADC0(GPIO26)
- J8 pad 2: Net-(J8-Pin_2) -> TMS_PIN
- J8 pad 3: Net-(J8-Pin_3) -> TDI/SWDIO_PIN
- J8 pad 4: Net-(J8-Pin_4) -> TDO_PIN
- L1 pad 2: Net-(IC1-SET) -> Net-(IC1-EN)
- R12 pad 1: Net-(IC2-XOUT) -> Net-(U5-GPIO10)
- R12 pad 2: Net-(U3-OSC2) -> SPI1_CLK0
- R17 pad 2: I2CSCL_ADC -> I2CSCL_EXT
- R18 pad 2: I2CSDA_ADC -> I2CSDA_EXT
- R23 pad 1: Net-(U4-ADDR) -> +3.3V_ADC
- R23 pad 2: GND -> SPI1_MISO
- R54 pad 1: TMS_PIN -> +3.3V_ADC
- R54 pad 2: Net-(J8-Pin_2) -> SPI1_MOSI
- R57 pad 1: TDI/SWDIO_PIN -> +3.3V_ADC
- R57 pad 2: Net-(J8-Pin_3) -> SPI1_CS0_N
- R58 pad 1: TDO_PIN -> +3.3V_ADC
- R58 pad 2: Net-(J8-Pin_4) -> SPI1_MOSI
- R60 pad 1: Net-(J8-Pin_3) -> +3.3V_ADC
- R60 pad 2: TDO_PIN -> SPI1_MISO
- R66 pad 1: ADC0(GPIO26) -> +3.3V_ADC
- R66 pad 2: Net-(J11-Pin_1) -> SPI1_CS1_N
- R7 pad 1: Net-(IC1-EN) -> Net-(IC1-SET)
- U3 pad 3: Net-(U3-OSC2) -> Net-(IC2-XOUT)
- U4 pad 1: Net-(U4-ADDR) -> SPI1_CLK0
- U4 pad 10: I2CSCL_ADC -> SPI1_MOSI
- U4 pad 2: unconnected-(U4-ALERT_RDY-Pad2) -> SPI1_CS0_N
- U4 pad 9: I2CSDA_ADC -> SPI1_MISO
- U5 pad 11: unconnected-(U5-GPIO8-Pad11) -> SPI1_MISO
- U5 pad 12: Net-(U5-GPIO9) -> unconnected-(U5-GPIO9-Pad12)
- U5 pad 13: unconnected-(U5-GPIO10-Pad13) -> Net-(U5-GPIO10)
- U5 pad 14: Net-(U5-GPIO11) -> SPI1_MOSI
- U5 pad 36: unconnected-(U5-GPIO24-Pad36) -> SPI1_CS1_N
- U5 pad 39: ADC1(GPIO27) -> unconnected-(U5-GPIO27_ADC1-Pad39)
- U5 pad 4: I2CSDA_ADC -> I2CSDA_EXT
- U5 pad 40: ADC2(GPIO28) -> unconnected-(U5-GPIO28_ADC2-Pad40)
- U5 pad 41: ADC3(GPIO28) -> unconnected-(U5-GPIO29_ADC3-Pad41)
- U5 pad 5: I2CSCL_ADC -> I2CSCL_EXT
- U5 pad 6: Net-(U5-GPIO4) -> SPI1_CS0_N
- U7 pad 1: Net-(U7-ADDR) -> SPI1_CLK0
- U7 pad 10: I2CSCL_ADC -> SPI1_MOSI
- U7 pad 2: unconnected-(U7-ALERT_RDY-Pad2) -> SPI1_CS1_N
- U7 pad 9: I2CSDA_ADC -> SPI1_MISO
Routing:
- net GND: track 1312.0 -> 1228.6 mm, vias 309 -> 341
- net SPI1_CLK0: track 0.00 -> 77.0 mm, vias 0 -> 1
- net SPI1_MISO: track 0.00 -> 64.1 mm, vias 0 -> 4
- net VBUS_EXT: track 0.00 -> 63.9 mm, vias 0 -> 4
- net SPI1_MOSI: track 0.00 -> 62.1 mm, vias 0 -> 4
- net ADC3(GPIO28): track 54.6 -> 0.00 mm, vias 3 -> 0
- net +3.3V_EXT: track 0.00 -> 53.5 mm, vias 0 -> 4
- net I2CSDA_ADC: track 52.3 -> 0.00 mm, vias 3 -> 0
- net I2CSCL_ADC: track 51.9 -> 0.00 mm, vias 3 -> 0
- net SPI1_CS0_N: track 0.00 -> 39.1 mm, vias 0 -> 1
- net SPI1_CS1_N: track 0.00 -> 37.8 mm, vias 0 -> 3
- net ADC1(GPIO27): track 31.0 -> 0.00 mm, vias 2 -> 0
- net ADC2(GPIO28): track 30.7 -> 0.00 mm, vias 2 -> 0
- net +3.3V_ADC: track 113.9 -> 92.6 mm, vias 5 -> 10
- net I2CSCL_EXT: track 0.00 -> 14.1 mm, vias 0 -> 1
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- added copper zone on B.Cu, net +3.3V_EXT
- added copper zone on In3.Cu, net +3.3V_EXT
- added copper zone on B.Cu, net VBUS_EXT
- added copper zone on In3.Cu, net VBUS_EXT
Other:
- board text added: "+"
- board text added: "+5V GND"
- board text added: "-"
- board text added: "ADC0 +3.3V"
- board text added: "I2CSDA I2CSCL"
- board text removed: "AD1"
- board text removed: "AD2"
- board text removed: "AD3"
- board text removed: "AD4"

Commit message: 2S commit
Routing:
- net GND: track 1228.6 -> 1258.6 mm, vias 341 -> 338
- net VCORE_FT2232H: track 44.5 -> 54.7 mm
- net TXD_PIN: track 51.5 -> 50.3 mm
- net RESET_N: track 85.8 -> 84.9 mm
- net +3.3V_EXT: track 53.5 -> 54.5 mm

Commit message: 3S commit
Parts:
- moved R64 1.18 mm to (157.6, 100.2), turned to -90 degrees
Routing:
- net GND: track 1258.6 -> 1244.2 mm, vias 338 -> 301
- net +3.3V_D: track 214.3 -> 215.6 mm
Other:
- board text added: "pi4 pi2 pi3 pi1"
- board text removed: "1"
- board text removed: "2"
- board text removed: "3"
- board text removed: "4"

Commit message: 3S commit
Routing:
- net GND: track 1244.2 -> 1251.1 mm
Other:
- board text added: "JLCJLCJLCJLC"
- board text removed: "JLCJLCJLC"
Changed lines of the file:
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@@
 		(tags "resistor handsolder")
 		(property "Reference" "R64"
-			(at 2.3125 -0.508 90)
+			(at 3.048 0.127 90)
 			(layer "B.SilkS")
 			(effects
@@
 		)
 	)
-	(gr_text "JLCJLCJLC"
+	(gr_text "JLCJLCJLCJLC"
 		(at 134.366 77.343 0)
 		(layer "F.SilkS")
@@
 	)
 	(segment
+		(start 138.057 74.414)
+		(end 138.049 74.422)
+		(width 0.1565)
+		(layer "B.Cu")
+		(net 13)
+	)
+	(segment
 		(start 118.491 97.155)
 		(end 118.5505 97.2145)
@@
 	)
 	(segment
+		(start 157.005 74.389)
+		(end 158.496 72.898)
+		(width 0.1565)
+		(layer "B.Cu")
+		(net 13)
+	)
+	(segment
 		(start 145.669 103.505)
 		(end 145.161 102.997)
@@
 	)
 	(segment
+		(start 136.906 73.279)
+		(end 136.779 73.279)
+		(width 0.1565)
+		(layer "B.Cu")
+		(net 13)
+	)
+	(segment
 		(start 126.492 99.441)
 		(end 126.492 99.187)
@@
 	)
 	(segment
+		(start 138.049 74.422)
+		(end 136.906 73.279)
+		(width 0.1565)
+		(layer "B.Cu")
+		(net 13)
+	)
+	(segment
 		(start 133.998 79.4525)
 		(end 133.998 80.2145)
@@
 	)
 	(segment
+		(start 138.408 74.414)
+		(end 138.057 74.414)
+		(width 0.1565)
+		(layer "B.Cu")
+		(net 13)
+	)
+	(segment
 		(start 145.161 102.997)
 		(end 145.161 102.489)
@@
 	)
 	(segment
+		(start 156.658 74.389)
+		(end 157.005 74.389)
+		(width 0.1565)
+		(layer "B.Cu")
+		(net 13)
+	)
+	(segment
 		(start 118.68325 92.64825)
 		(end 118.68325 93.208453)
@@
 	)
 	(segment
+		(start 133.408 74.414)
+		(end 132.961 74.414)
+		(width 0.1565)
+		(layer "B.Cu")
+		(net 13)
+	)
+	(segment
+		(start 131.826 73.279)
+		(end 131.699 73.279)
+		(width 0.1565)
+		(layer "B.Cu")
+		(net 13)
+	)
+	(segment
 		(start 148.316 94.267)
 		(end 143.985 94.267)
@@
 	)
 	(segment
+		(start 132.961 74.414)
+		(end 131.826 73.279)
+		(width 0.1565)
+		(layer "B.Cu")
+		(net 13)
+	)
+	(segment
 		(start 138.557 108.012)
 		(end 138.557 107.442)
@@
 	)
 	(segment
+		(start 158.496 72.898)
+		(end 158.496 72.771)
+		(width 0.1565)
+		(layer "B.Cu")
+		(net 13)
+	)
+	(segment
 		(start 141.732 110.236)
 		(end 141.478 110.49)
@@
 		(layer "B.Cu")
 		(hatch edge 0.5)
+		(connect_pads
+			(clearance 0)
+		)
+		(min_thickness 0.25)
+		(filled_areas_thickness no)
+		(keepout
+			(tracks not_allowed)
+			(vias not_allowed)
+			(pads not_allowed)
+			(copperpour not_allowed)
+			(footprints allowed)
+		)
+		(placement
+			(enabled no)
+			(sheetname "JTAG Select")
+		)
+		(fill
+			(thermal_gap 0.5)
+			(thermal_bridge_width 0.5)
+		)
+		(polygon
+			(pts
+				(xy 146.539857 80.264) (xy 146.539857 80.772) (xy 146.177 81.026) (xy 145.923 81.026) (xy 145.923 80.264)
+			)
+		)
+	)
+	(zone
+		(net 0)
+		(net_name "")
+		(layer "B.Cu")
+		(hatch edge 0.5)
 		(connect_pads yes
 			(clearance 0)
@@
 		(polygon
 			(pts
-				(xy 126.637143 77.216) (xy 126.854857 77.47) (xy 126.854857 78.105) (xy 125.73 78.105) (xy 125.73 77.343)
+				(xy 126.637143 77.216) (xy 127.254 77.47) (xy 127.235857 78.105) (xy 125.73 78.105) (xy 125.73 77.343)
 				(xy 125.984 77.216)
 			)
