File: FT2232H_EVB.kicad_pcb (KiCad board)
At the start: 6 copper layers, 50 x 50 mm, 214 parts, among them IC1 MT9700, IC2 SL2.1s, IC3 W25Q16JVUXIQ, IC4 LCMXO2-1200HC-4SG32I, J1 GT-USB-7010ASV, J10 Conn_01x04, J11 Conn_02x03_Odd_Even, J13 Conn_02x01, J2 WJ126V-5.0-2P, J3 WJ126V-5.0-2P, J4 WJ126V-5.0-2P, J5 WJ126V-5.0-2P, J6 Conn_02x03_Odd_Even, J7 Conn_02x03_Odd_Even, J8 Conn_02x03_Odd_Even, J9 Conn_02x03_Odd_Even, SW1 DSWB03LHGET, U1 RT5752BHGJ5, U10 RQ12000160, U11 TMUX1574DYYR, U12 TMUX1574DYYR, U2 TLV803SDBZR, U3 RQ12000160, U4 ADS1118IDGSR, U5 RP2040, U6 RQ12000160, U7 ADS1118IDGSR, U8 FT2232HL, U9 93LC56BT-I

Commit message: Mass Production2 commit
Routing:
- net GND: track 1270.5 -> 1284.8 mm, vias 299 -> 363
- net Net-(J2-Pin_1): track 5.10 -> 4.21 mm

Commit message: Mass Production2 commit
Parts:
- removed C8: 10p, Capacitor_SMD:C_0201_0603Metric_Pad0.64x0.40mm_HandSolder
- moved R8 7.02 mm to (126.4, 100.4), turned to 90 degrees
- moved R4 6.65 mm to (125.4, 98.5)
- moved L3 4.11 mm to (127.5, 93.8), turned to 180 degrees
- moved C5 3.46 mm to (123.5, 94.6), turned to 180 degrees
- moved C2 0.97 mm to (124.4, 98.7), turned to 90 degrees
- moved U1 0.89 mm to (127.5, 97.5), turned to -90 degrees
- moved C3 0.86 mm to (128.8, 101.8), turned to 0 degrees
- moved C4 0.86 mm to (128.8, 100.3), turned to 0 degrees
Routing:
- net GND: track 1284.8 -> 1265.0 mm, vias 363 -> 365
- net +3.3V: track 35.2 -> 27.9 mm
- net +3.3V_D: track 215.6 -> 221.5 mm
- net Net-(U1-EN): track 10.6 -> 9.04 mm
- removed copper zone on B.Cu, net Net-(U1-EN)

Commit message: Mass Production2 commit
Parts:
- removed R62: 0, Resistor_SMD:R_0201_0603Metric_Pad0.64x0.40mm_HandSolder
Connections:
- U8 pad 3: Net-(U8-OSCO) -> Net-(U10-OSC2)
Routing:
- net GND: track 1265.0 -> 1286.1 mm, vias 365 -> 367
- net Net-(U10-OSC2): track 3.83 -> 9.41 mm
- net Net-(U8-OSCO): track 4.20 -> 0.00 mm
- net Net-(IC2-XOUT): track 8.19 -> 8.73 mm
