File: FT2232H_EVB.kicad_pcb (KiCad board)
At the start: 6 copper layers, 50 x 50 mm, 212 parts, among them IC1 MT9700, IC2 SL2.1s, IC3 W25Q16JVUXIQ, IC4 LCMXO2-1200HC-4SG32I, J1 GT-USB-7010ASV, J10 Conn_01x04, J11 Conn_02x03_Odd_Even, J13 Conn_02x01, J2 WJ126V-5.0-2P, J3 WJ126V-5.0-2P, J4 WJ126V-5.0-2P, J5 WJ126V-5.0-2P, J6 Conn_02x03_Odd_Even, J7 Conn_02x03_Odd_Even, J8 Conn_02x03_Odd_Even, J9 Conn_02x03_Odd_Even, SW1 DSWB03LHGET, U1 RT5752BHGJ5, U10 RQ12000160, U11 TMUX1574DYYR, U12 TMUX1574DYYR, U2 TLV803SDBZR, U3 RQ12000160, U4 ADS1118IDGSR, U5 RP2040, U6 RQ12000160, U7 ADS1118IDGSR, U8 FT2232HL, U9 93LC56BT-I

Commit message: Mass Production2 commit
Parts:
- J13: value Conn_02x01 -> PH-2A; footprint Connector_PinHeader_2.54mm:PinHeader_2x01_P2.54mm_Vertical -> Connector_JST:JST_PH_B2B-PH-K_1x02_P2.00mm_Vertical
- moved D2 1.23 mm to (113.5, 89.7)
- moved J13 1.23 mm to (114.5, 85.1)
- moved R5 1.22 mm to (115.5, 89.7)
- moved C75 1.08 mm to (115.4, 83.7)
Routing:
- net VBUS_EXT: track 63.9 -> 61.6 mm
- net Net-(D1-A1): track 60.7 -> 59.5 mm
- net GND: track 1286.1 -> 1285.2 mm, vias 367 -> 359
- added copper zone on In5.Cu, net +1.1V_MCU
- added copper zone on In5.Cu, net +3.3V_ADC
- added copper zone on In5.Cu, net +3.3V_A_FT2232H
- added copper zone on In5.Cu, net +3.3V_D
- added copper zone on In4.Cu, net +3.3V_EXT
- added copper zone on In5.Cu, net +3.3V_FT2232H
- added copper zone on In5.Cu, net GND
- added copper zone on In6.Cu, net GND
- added copper zone on In5.Cu, net VBUS
- added copper zone on In4.Cu, net VBUS_EXT
- added copper zone on In5.Cu, net VCORE_FT2232H
- removed copper zone on In4.Cu, net +1.1V_MCU
- removed copper zone on In4.Cu, net +3.3V_ADC
- removed copper zone on In4.Cu, net +3.3V_A_FT2232H
- removed copper zone on In4.Cu, net +3.3V_D
- removed copper zone on In3.Cu, net +3.3V_EXT
- removed copper zone on In4.Cu, net +3.3V_FT2232H
- removed copper zone on In4.Cu, net VBUS
- removed copper zone on In3.Cu, net VBUS_EXT
- removed copper zone on In4.Cu, net VCORE_FT2232H
Other:
- copper layers 6 -> 8

Commit message: Mass Production2 commit
Routing:
- net GND: track 1285.2 -> 1275.8 mm, vias 359 -> 376
- net Net-(U10-OSC2): track 9.41 -> 11.1 mm
- net /FT2232H_N: track 7.81 -> 7.02 mm
